File: rucheb.kicad_sch (KiCad schematic)
At the start: 28 parts, among them IC1 CN3791, IC9 FS312F-G, J1 Conn_01x02, Q1 AO3401A, Q8 FS8205

Commit message: update
Parts:
- D1, D3, D4: footprint LED_SMD:LED_0603_1608Metric_Castellated -> LED_SMD:LED_0603_1608Metric_Pad1.05x0.95mm_HandSolder
