File: Open_beehive_scale_V0.5.kicad_pcb (KiCad board)
At the start: 2 copper layers, 92.8 x 99.9 mm, 197 parts, among them IC1 CN3791, IC2 MAX17048G+, IC4 SHT41-AD1B-R3, IC5 HX711, IC6 HX711, IC7 HX711, IC8 HX711, IC9 FS312F-G, J1 Conn_01x02, J10 Conn_01x04, J11 Conn_01x04, J12 Conn_01x04, J13 Micro_SD_Card, J14 Conn_01x03, J15 Conn_01x04, J16 Conn_01x04, J17 Conn_01x04, J18 Conn_01x04, J19 Conn_01x02, J2 Conn_01x04, J20 USB_C_Receptacle_USB2.0 USB41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, J21 Conn_01x02, J22 Conn_01x08, J23 USB_C_Receptacle_USB2.0 USB41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, J3 Conn_01x03, J4 Conn_01x02, J5 Conn_01x04, J6 Conn_01x02, J7 Conn_01x02, J8 Conn_01x03, J9 Conn_01x03, Q1 AO3401A, Q2 MMBT4403, Q3 MMBT4403, Q4 MMBT4403, Q5 MMBT4403, Q6 UMH3N, Q7 DMG2301L, Q8 FS8205, SW1 SW_Push, SW2 SW_Push, U1 CP2102N-A02-GQFN24, U2 MS5611-01BA, U3 XC6220B331MR, U4 TCA9548APWR, U5 XC6220B331MR, U7 1043, U8 ESP32-S3-WROOM-2, U9 XC6220B331MR

Commit message: update
Parts:
- removed C55: 4.7µF, Capacitor_SMD:C_0805_2012Metric
- removed C56, C65: 0.1µF, Capacitor_SMD:C_0603_1608Metric
- removed D13, D8, D9: SP1003-01DTG, Empreintes:SODFL1406X65N
- removed D7: LED, LED_SMD:LED_0603_1608Metric
- removed J14, J9: Conn_01x03, Connector_JST:JST_PH_B3B-PH-K_1x03_P2.00mm_Vertical
- removed J19: Conn_01x02, Connector_JST:JST_PH_B2B-PH-K_1x02_P2.00mm_Vertical
- removed J23: USB_C_Receptacle_USB2.0 USB4105-GF-A, Empreintes:TYPE-C-31-M-12
- removed Q6: UMH3N, Package_TO_SOT_SMD:SOT-363_SC-70-6
- removed R11, R54: 10K, Resistor_SMD:R_0603_1608Metric
- removed R41: 22.1K, Resistor_SMD:R_0603_1608Metric
- removed R44: 47.5k, Resistor_SMD:R_0603_1608Metric
- removed R47: 1K, Resistor_SMD:R_0603_1608Metric
- removed R56: 1M, Resistor_SMD:R_0603_1608Metric
- removed R57, R58: 5.1K, Resistor_SMD:R_0603_1608Metric
- removed R9: 4.7K, Resistor_SMD:R_0603_1608Metric
- removed S1: RB231X2, Empreintes:RB231X2
- removed SW2: SW_Push, Empreintes:PTS636SL43SMTRLFS
- removed U1: CP2102N-A02-GQFN24, Package_DFN_QFN:QFN-24-1EP_4x4mm_P0.5mm_EP2.6x2.6mm
- J3, J8: value Conn_01x03 -> Conn_01x02; footprint Connector_JST:JST_PH_B3B-PH-K_1x03_P2.00mm_Vertical -> Connector_JST:JST_PH_B2B-PH-K_1x02_P2.00mm_Vertical
- moved J5 74.8 mm to (134.6, 130.2), turned to 90 degrees
- moved J8 54.3 mm to (136.1, 115.7)
- moved J21 40.8 mm to (128.0, 73.3), turned to 90 degrees
- moved C12 39.7 mm to (165.2, 75.3)
- moved C13 39.7 mm to (160.4, 75.3)
- moved C14 39.7 mm to (158.7, 75.4)
- moved FB1 39.7 mm to (162.8, 76.2)
- moved U2 39.7 mm to (155.6, 74.3)
- moved R43 38.1 mm to (126.3, 78.8)
- moved J3 37.8 mm to (136.1, 108.6)
- moved SW1 34.5 mm to (144.9, 111.0), turned to 90 degrees
- moved C57 11.1 mm to (129.2, 79.2)
- moved C58 11.1 mm to (131.1, 77.5)
- moved R48 10.5 mm to (145.5, 121.0), turned to 180 degrees
- moved J11 10.5 mm to (103.9, 89.2)
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Connections:
- C17 pad 1: VCC_GPS -> VCC_MODEM
- C18 pad 1: VCC_GPS -> VCC_MODEM
- D11 pad 1: USBD_P -> USB_D+
- D12 pad 1: USBD_N -> USB_D-
- J20 pad A6: USBD_P -> USB_D+
- J20 pad A7: USBD_N -> USB_D-
- J20 pad B6: USBD_P -> USB_D+
- J20 pad B7: USBD_N -> USB_D-
- J22 pad 8: VBAT -> VCC_MODEM
- J3 pad 1: VCC -> wifi
- J3 pad 2: DS18b20 -> GND
- J8 pad 1: VCC -> Led
- J8 pad 2: DS18b20 -> GND
- R10 pad 2: INT1 -> wifi
- U3 pad 3: Start_GPS -> Start_Modem
- U3 pad 5: VCC_GPS -> VCC_MODEM
- U8 pad 15: CLK4 -> unconnected-(U8-GPIO3/TOUCH3/ADC1_CH2-Pad15)
- U8 pad 17: PWRKEY -> UART_RXD
- U8 pad 18: UART_RXD -> UART_TXD
- U8 pad 19: UART_TXD -> DAT4
- U8 pad 20: Tilt_led_alarm -> CLK4
- U8 pad 23: DS18b20 -> DAT3
- U8 pad 24: CLK2 -> unconnected-(U8-GPIO47/SPICLK_P/SUBSPICLK_P_DIFF-Pad24)
- U8 pad 31: unconnected-(U8-GPIO38/FSPIWP/SUBSPIWP-Pad31) -> Start_Modem
- U8 pad 32: SDO-MISO-D10 -> DAT2
- U8 pad 33: CMD-MOSI-D8 -> CLK2
- U8 pad 34: CLK-SCK-D9 -> unconnected-(U8-MTDI/GPIO41/CLK_OUT1-Pad34)
- U8 pad 35: SD3-CS-D7 -> CLK3
- U8 pad 36: UORXD -> unconnected-(U8-U0RXD/GPIO44/CLK_OUT2-Pad36)
- U8 pad 37: UOTXD -> unconnected-(U8-U0TXD/GPIO43/CLK_OUT1-Pad37)
- U8 pad 38: DAT4 -> DAT1
- U8 pad 39: Start_Modem -> CLK1
- U8 pad 4: DAT2 -> Led
- U8 pad 5: DAT1 -> CLK-SCK-D9
- U8 pad 6: CLK3 -> CMD-MOSI-D8
- U8 pad 7: DAT3 -> SDO-MISO-D10
- U8 pad 8: CLK1 -> SD3-CS-D7
- U8 pad 9: INT1 -> wifi
Routing:
- net USB_D-: track 0.00 -> 102.8 mm, vias 0 -> 2
- net USB_D+: track 0.00 -> 100.6 mm
- net DS18b20: track 77.1 -> 0.00 mm, vias 3 -> 0
- net DTR_E: track 0.00 -> 74.9 mm
- net UART_RXD: track 0.00 -> 65.1 mm, vias 0 -> 2
- net PWRKEY: track 0.00 -> 63.4 mm, vias 0 -> 2
- net UART_TXD: track 0.00 -> 63.0 mm, vias 0 -> 2
- net IO0: track 58.3 -> 0.00 mm, vias 2 -> 0
- net Start_Modem: track 0.00 -> 51.3 mm, vias 0 -> 2
- net UORXD: track 49.0 -> 0.00 mm, vias 2 -> 0
- net UOTXD: track 46.3 -> 0.00 mm, vias 3 -> 0
- net CLK3: track 2.60 -> 39.8 mm, vias 0 -> 2
- net SDA: track 90.8 -> 122.2 mm
- net +3V3: track 148.8 -> 118.4 mm, vias 9 -> 6
- net SCL: track 90.2 -> 119.1 mm, vias 6 -> 5
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Other:
- outline, holes or cut-outs redrawn
- board text removed: "1-DAT-2"
- board text removed: "3-DAT-4"
- board text removed: "DS18b20 1 to 4"
- board text removed: "T I L T"
- board text removed: "Tilt alarm"

Commit message: update
Parts:
- added Q6: PMBT2222A,215, Empreintes:PMBT2222A215, F.Cu at (136.2, 116.1)
- C15: footprint Capacitor_SMD:C_0603_1608Metric -> Capacitor_SMD:C_0805_2012Metric
- C16: footprint Capacitor_SMD:C_0805_2012Metric -> Capacitor_SMD:C_0603_1608Metric
- D1, D3, D4: footprint LED_SMD:LED_0603_1608Metric_Castellated -> LED_SMD:LED_0603_1608Metric_Pad1.05x0.95mm_HandSolder
- J5: footprint Connector_JST:JST_PH_B4B-PH-K_1x04_P2.00mm_Vertical -> Empreintes:1989764
- J8: footprint Connector_JST:JST_PH_B2B-PH-K_1x02_P2.00mm_Vertical -> Empreintes:1989748
- moved G*** 26.2 mm to (134.3, 127.2)
- moved J5 22.4 mm to (152.3, 143.9), turned to -90 degrees
- moved J3 17.2 mm to (121.4, 99.8), turned to 0 degrees
- moved FID2 8.06 mm to (173.5, 77.2)
- moved J8 4.20 mm to (136.3, 111.5)
- moved R10 0.13 mm to (128.2, 114.7)
Connections:
- J8 pad 1: Led -> Net-(J8-Pin_1)
- J8 pad 2: GND -> VCC
Routing:
- net Led: track 0.00 -> 46.9 mm, vias 0 -> 2
- net wifi: track 0.00 -> 40.9 mm, vias 0 -> 1
- net SDA: track 122.2 -> 133.4 mm, vias 4 -> 8
- net SCL: track 119.1 -> 127.4 mm, vias 5 -> 7
- net Start_Modem: track 51.3 -> 57.4 mm
- net Net-(J8-Pin_1): track 0.00 -> 3.67 mm
- net VCC: track 363.2 -> 362.6 mm
- net GND: vias 184 -> 185
Other:
- outline, holes or cut-outs redrawn
- board text added: "Led"
- board text added: "Opensource connected hive V0.5 by Ratamuse"
- board text added: "Wifi"
- board text removed: "Boot"
- board text removed: "Opensource connected hive V0.4 by Ratamuse"
- board text removed: "Reset"

Commit message: Update
Parts:
- added C11: 0.1µF, Capacitor_SMD:C_0603_1608Metric, F.Cu at (162.7, 142.0)
- added C20: 0.1µF, Capacitor_SMD:C_0603_1608Metric, F.Cu at (162.0, 145.7)
- added C21: 0.150µF, Capacitor_SMD:C_0603_1608Metric, F.Cu at (162.7, 148.0)
- added C55: 0.150µF, Capacitor_SMD:C_0603_1608Metric, F.Cu at (169.4, 145.1)
- added C6: 1µF, Capacitor_SMD:C_0603_1608Metric, F.Cu at (161.2, 142.0)
- added IC3: LTC2954CTS8-1#TRMPBF, Empreintes:SOT65P280X100-8N, F.Cu at (166.1, 144.7)
- added J9: Conn_01x02, Empreintes:1725656, F.Cu at (155.2, 144.3)
- added R41: 5.1K, Resistor_SMD:R_0603_1608Metric, F.Cu at (162.0, 144.2)
- added R42: 10K, Resistor_SMD:R_0603_1608Metric, F.Cu at (167.4, 148.0)
- J11, J12, J17, J18: footprint Connector_JST:JST_PH_B4B-PH-K_1x04_P2.00mm_Vertical -> Empreintes:1725672
- J3: footprint Connector_JST:JST_PH_B2B-PH-K_1x02_P2.00mm_Vertical -> Empreintes:1725656
- J5: footprint Empreintes:1989764 -> Empreintes:1725672
- J8: footprint Empreintes:1989748 -> Empreintes:1725656
- moved J5 67.0 mm to (168.3, 78.8), turned to 0 degrees
- moved FID2 21.4 mm to (171.5, 98.4)
- moved Q6 13.0 mm to (129.6, 105.0), turned to 180 degrees
- moved J8 6.13 mm to (131.1, 108.3), turned to -90 degrees
- moved G*** 2.11 mm to (132.8, 128.6)
- moved R7 1.94 mm to (138.6, 129.7)
- moved R8 1.94 mm to (139.4, 127.9)
- moved J17 0.80 mm to (89.7, 89.2)
- moved J12 0.75 mm to (89.7, 99.9)
Connections:
- J22 pad 3: Vref -> VCC_MODEM
- J5 pad 2: SCL -> SDA
- J5 pad 3: SDA -> SCL
- U8 pad 11: Start_modules -> DTR_E
- U8 pad 12: DTR_E -> Start_modules
- U8 pad 24: unconnected-(U8-GPIO47/SPICLK_P/SUBSPICLK_P_DIFF-Pad24) -> CLK3
- U8 pad 25: unconnected-(U8-GPIO48/SPICLK_N/SUBSPICLK_N_DIFF-Pad25) -> PWRKEY
- U8 pad 35: CLK3 -> unconnected-(U8-MTMS/GPIO42-Pad35)
- U9 pad 3: +5V -> CE
Routing:
- net +3V3: track 118.8 -> 145.0 mm, vias 6 -> 8
- net Start_modules: track 39.4 -> 60.7 mm
- net CE: track 0.00 -> 20.2 mm, vias 0 -> 2
- net Led: track 46.9 -> 27.8 mm, vias 2 -> 0
- net VCC_MODEM: track 17.2 -> 35.3 mm
- net PWRKEY: track 63.4 -> 80.1 mm
- net SDA: track 133.4 -> 149.0 mm, vias 8 -> 7
- net CLK3: track 39.8 -> 24.4 mm, vias 2 -> 0
- net SCL: track 127.4 -> 141.9 mm
- net +5V: track 60.4 -> 74.6 mm, vias 2 -> 3
- net Net-(J9-Pin_1): track 0.00 -> 5.97 mm
- net Net-(IC3-ONT): track 0.00 -> 3.74 mm
- net DTR_E: track 74.9 -> 78.6 mm
- net Net-(IC3-~{PB}): track 0.00 -> 3.58 mm
- net USB_D+: track 100.6 -> 97.8 mm
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
Commit message: update
Parts:
- J22: footprint Connector_PinHeader_2.54mm:PinHeader_1x08_P2.54mm_Vertical -> Empreintes:Sim8070G
- moved G*** 57.6 mm to (141.9, 85.2)
- moved J22 22.5 mm to (122.0, 136.1), turned to 180 degrees
- moved G*** 16.3 mm to (150.0, 121.8)
Routing:
- net VCC_MODEM: track 35.3 -> 30.7 mm
- net USB_D+: track 97.8 -> 100.3 mm
- net GND: track 52.0 -> 50.3 mm, vias 196 -> 225
- net UART_RXD: track 64.1 -> 62.4 mm
- net UART_TXD: track 62.1 -> 60.7 mm
- net PWRKEY: track 80.1 -> 78.8 mm
- net Start_modules: track 60.7 -> 60.2 mm
Other:
- outline, holes or cut-outs redrawn

Commit message: update
Parts:
- added JP1: Jumper_2_Open, Jumper:SolderJumper-2_P1.3mm_Open_RoundedPad1.0x1.5mm, F.Cu at (148.3, 121.8)
- J21: footprint Connector_JST:JST_PH_B2B-PH-K_1x02_P2.00mm_Vertical -> Empreintes:1725656
- moved G*** 67.9 mm to (119.5, 57.6)
- moved J21 27.8 mm to (142.0, 49.3), turned to 180 degrees
- moved U3 27.3 mm to (148.0, 110.1)
- moved C15 27.3 mm to (150.9, 111.8)
- moved C17 27.3 mm to (145.2, 111.8)
- moved C16 27.3 mm to (152.5, 112.0)
- moved C18 27.3 mm to (143.3, 111.9)
- moved G*** 26.9 mm to (144.9, 104.6)
- moved C3 26.5 mm to (133.0, 134.1)
- moved C2 26.4 mm to (134.7, 133.9)
- moved C1 26.4 mm to (115.2, 136.6)
- moved C12 26.4 mm to (177.9, 52.0)
- moved C13 26.4 mm to (173.0, 52.0)
- moved C21 26.4 mm to (175.3, 124.8)
- moved C25 26.4 mm to (181.0, 82.7)
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Routing:
- net VCC_MODEM: track 30.7 -> 47.8 mm
- net GND: track 50.3 -> 66.6 mm, vias 225 -> 286
- net +5V: track 74.6 -> 81.8 mm, vias 3 -> 4
- net SDA: track 149.0 -> 146.1 mm, vias 7 -> 6
- net Start_modules: track 60.2 -> 57.8 mm
- net Rain_gauge: track 24.5 -> 26.5 mm
- net VCC: track 365.0 -> 363.2 mm
- net SCL: track 141.9 -> 140.2 mm
- net Start_Modem: track 57.7 -> 56.8 mm
- net PWRKEY: track 78.8 -> 79.7 mm
- net +3V3: track 145.0 -> 144.2 mm, vias 8 -> 7
- net UART_RXD: track 62.4 -> 63.2 mm
- net SC3: track 31.5 -> 30.7 mm
- net wifi: track 40.9 -> 40.2 mm
- net UART_TXD: track 60.7 -> 61.3 mm
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
Commit message: update
Parts:
- removed the G*** at (177.3, 68.3)
- removed JP1: Jumper_2_Open, Jumper:SolderJumper-2_P1.3mm_Open_RoundedPad1.0x1.5mm
- added C56: 0.010µF, Capacitor_SMD:C_0603_1608Metric, F.Cu at (180.8, 119.0)
- added JP2: Jumper_2_Open, Jumper:SolderJumper-2_P1.3mm_Open_RoundedPad1.0x1.5mm, B.Cu at (179.6, 118.2)
- added JP3: Jumper_2_Open, Jumper:SolderJumper-2_P1.3mm_Open_RoundedPad1.0x1.5mm, F.Cu at (135.7, 111.3)
- added JP4: Jumper_2_Open, Jumper:SolderJumper-2_P1.3mm_Open_RoundedPad1.0x1.5mm, F.Cu at (148.4, 121.8)
- added Q10: AO3400, Package_TO_SOT_SMD:SOT-23, F.Cu at (151.0, 138.2)
- added R9: 100K, Resistor_SMD:R_0603_1608Metric, F.Cu at (180.8, 117.5)
- moved J4 53.1 mm to (116.3, 118.7), turned to 180 degrees
- moved G*** 11.3 mm to (166.2, 66.0)
- moved G*** 5.26 mm to (164.8, 93.8)
- moved G*** 4.78 mm to (141.5, 101.3)
- moved C64 2.00 mm to (156.0, 139.8)
- moved IC9 2.00 mm to (156.5, 137.5)
- moved Q8 2.00 mm to (155.8, 134.4)
- moved R52 2.00 mm to (160.4, 137.5)
- moved R53 2.00 mm to (159.1, 139.7)
- moved FID1 0.94 mm to (116.9, 53.4)
- moved J22 0.39 mm to (134.6, 113.3)
- moved C55 0.32 mm to (182.4, 121.9)
Connections:
- net Sensor_VN_IO39 renamed Net-(IC3-~{INT})
- IC3 pad 8: PS_HOLD_IO33 -> Net-(IC3-~{KILL})
- J21 pad 1: Rain_gauge -> GND
- J21 pad 2: GND -> Rain_gauge
- J22 pad 8: VCC_MODEM -> Net-(J22-Pin_8)
- U7 pad 2: VBAT- -> Net-(U7--)
Routing:
- net VBAT: track 63.5 -> 124.3 mm
- net wifi: track 40.2 -> 100.5 mm, vias 1 -> 4
- net Net-(U7--): track 0.00 -> 50.8 mm, vias 0 -> 2
- net VBAT-: track 61.7 -> 14.7 mm, vias 2 -> 0
- net Net-(J22-Pin_8): track 0.00 -> 23.8 mm, vias 0 -> 1
- net +3V3: track 144.2 -> 158.2 mm
- net VCC_MODEM: track 47.8 -> 34.8 mm
- net GND: track 66.6 -> 76.4 mm, vias 286 -> 276
- net Net-(IC3-~{INT}): track 1.53 -> 7.78 mm, vias 0 -> 1
- net Net-(IC3-~{KILL}): track 0.00 -> 3.00 mm
- net SDA: track 146.1 -> 143.9 mm
- net Net-(J16-Pin_2): track 22.9 -> 21.5 mm
- net Rain_gauge: track 26.5 -> 25.4 mm
- net CLK3: track 24.4 -> 25.1 mm
- net DAT3: track 26.7 -> 27.3 mm
Other:
- outline, holes or cut-outs redrawn
- board text added: "+3V3"
- board text added: "Fuel gauge"
- board text added: "Modem VBat"
- board text added: "ON/OFF"
- board text added: "Opensource connected hive V0.5 by Ratamuse NB-Iot version"
- board text added: "Vcc"
- board text added: "Vcc_modem"
- board text removed: "Opensource connected hive V0.5 by Ratamuse"
