File: Open_beehive_scale_V0.5.kicad_pcb (KiCad board)
At the start: 2 copper layers, 92.8 x 99.9 mm, 188 parts, among them IC1 CN3791, IC2 MAX17048G+, IC3 LTC2954CTS8-1#TRMPBF, IC4 SHT41-AD1B-R3, IC5 HX711, IC6 HX711, IC7 HX711, IC8 HX711, IC9 FS312F-G, J1 Conn_01x02, J10 Conn_01x04, J11 Conn_01x04, J12 Conn_01x04, J13 Micro_SD_Card, J15 Conn_01x04, J16 Conn_01x04, J17 Conn_01x04, J18 Conn_01x04, J2 Conn_01x04, J20 USB_C_Receptacle_USB2.0 USB41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, J21 Conn_01x02, J22 Conn_01x08, J3 Conn_01x02, J4 Conn_01x02, J5 Conn_01x04, J6 Conn_01x02, J7 Conn_01x02, J8 Conn_01x02, J9 Conn_01x02, Q1 AO3401A, Q10 AO3400, Q2 MMBT4403, Q3 MMBT4403, Q4 MMBT4403, Q5 MMBT4403, Q6 PMBT2222A,215, Q7 DMG2301L, Q8 FS8205, SW1 SW_Push, U2 MS5611-01BA, U3 XC6220B331MR, U4 TCA9548APWR, U5 XC6220B331MR, U7 1043, U8 ESP32-S3-WROOM-2, U9 XC6220B331MR

Commit message: update
Parts:
- added R44: 100k, Resistor_SMD:R_0603_1608Metric, F.Cu at (164.1, 129.0)
- J20: value USB_C_Receptacle_USB2.0 USB4105-GF-A -> USB_C_Receptacle_USB2.0 USB4105-GF-A
Routing:
- net GND: track 76.4 -> 72.6 mm, vias 276 -> 277
- net CE: track 20.2 -> 23.2 mm
- net +5V: track 81.3 -> 83.7 mm, vias 4 -> 5
