File: Open_beehive_scale_V0.5.kicad_sch (KiCad schematic)
At the start: 43 parts, among them IC2 MAX17048G+, IC4 SHT41-AD1B-R3, J13 Micro_SD_Card, J19 Conn_01x02, J21 Conn_01x02, J22 Conn_01x08, U2 MS5611-01BA, U3 XC6220B331MR, U5 XC6220B331MR, U9 XC6220B331MR

Commit message: update
Parts:
- removed D7: LED, LED_SMD:LED_0603_1608Metric, symbol Device:LED
- removed J19: Conn_01x02, Connector_JST:JST_PH_B2B-PH-K_1x02_P2.00mm_Vertical, symbol Connector_Generic:Conn_01x02
- removed R11: 10K, Resistor_SMD:R_0603_1608Metric, symbol Device:R
- removed S1: RB231X2, Empreintes:RB231X2, symbol RB231X2:RB231X2
- added J3: Conn_01x02, Connector_JST:JST_PH_B2B-PH-K_1x02_P2.00mm_Vertical, symbol Connector_Generic:Conn_01x02
Connections:
- net GND: now also J3.2 (Pin_2)
- net VBAT: no longer J22.8 (Pin_8)
- net INT1 renamed wifi
- net wifi: now also J3.1 (Pin_1)
- net Start_GPS renamed Start_Modem
- net VCC_GPS renamed VCC_MODEM
- net VCC_MODEM: now also J22.8 (Pin_8)
Other:
- note added: "Wifi connect push button"
- note removed: "External RESET push button"
- note removed: "Tilt sensor (suspicious mouvement alarm)"
- moved on the sheet: R10

Commit message: Update
Parts:
- added JP1: SolderJumper_2_Open, symbol Jumper:SolderJumper_2_Open
- J3: footprint Connector_JST:JST_PH_B2B-PH-K_1x02_P2.00mm_Vertical -> Empreintes:1725656
Connections:
- net Vref is gone; now on net VCC_MODEM: J22.3 (Pin_3)
- net +5V: no longer U9.3 (CE)
- new net CE: U9.3 (CE)
Changed lines of the file:
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@@
 	)
 	(junction
+		(at 104.902 167.64)
+		(diameter 0)
+		(color 0 0 0 0)
+	)
+	(junction
 		(at 76.2 39.37)
 		(diameter 0)
@@
 	)
 	(junction
-		(at 146.05 21.59)
-		(diameter 0)
-		(color 0 0 0 0)
-	)
-	(junction
 		(at 45.72 167.64)
 		(diameter 0)
@@
 	(wire
 		(pts
-			(xy 102.87 167.64) (xy 107.95 167.64)
+			(xy 102.87 167.64) (xy 104.902 167.64)
 		)
 		(stroke
@@
 	(wire
 		(pts
-			(xy 45.72 167.64) (xy 63.5 167.64)
-		)
-		(stroke
-			(width 0)
-			(type default)
-		)
-	)
-	(wire
-		(pts
 			(xy 248.92 97.79) (xy 256.54 97.79)
 		)
@@
 	(wire
 		(pts
-			(xy 146.05 21.59) (xy 148.59 21.59)
-		)
-		(stroke
-			(width 0)
-			(type default)
-		)
-	)
-	(wire
-		(pts
 			(xy 129.54 21.59) (xy 130.81 21.59)
 		)
@@
 	(wire
 		(pts
-			(xy 146.05 26.67) (xy 148.59 26.67)
+			(xy 45.72 167.64) (xy 63.5 167.64)
 		)
 		(stroke
@@
 	(wire
 		(pts
+			(xy 104.902 161.798) (xy 107.95 161.798)
+		)
+		(stroke
+			(width 0)
+			(type default)
+		)
+	)
+	(wire
+		(pts
 			(xy 251.46 106.68) (xy 266.7 106.68)
 		)
@@
 	(wire
 		(pts
-			(xy 146.05 21.59) (xy 146.05 26.67)
+			(xy 63.5 81.28) (xy 68.58 81.28)
 		)
 		(stroke
@@
 	(wire
 		(pts
-			(xy 63.5 81.28) (xy 68.58 81.28)
+			(xy 101.6 36.83) (xy 101.6 39.37)
 		)
 		(stroke
@@
 	(wire
 		(pts
-			(xy 101.6 36.83) (xy 101.6 39.37)
+			(xy 147.574 26.67) (xy 148.59 26.67)
 		)
 		(stroke
@@
 	(wire
 		(pts
+			(xy 104.902 167.64) (xy 107.95 167.64)
+		)
+		(stroke
+			(width 0)
+			(type default)
+		)
+	)
+	(wire
+		(pts
 			(xy 53.34 58.42) (xy 63.5 58.42)
 		)
@@
 	(wire
 		(pts
+			(xy 104.902 161.798) (xy 104.902 167.64)
+		)
+		(stroke
+			(width 0)
+			(type default)
+		)
+	)
+	(wire
+		(pts
 			(xy 102.87 172.72) (xy 102.87 167.64)
 		)
@@
 	(wire
 		(pts
-			(xy 140.97 21.59) (xy 146.05 21.59)
+			(xy 140.97 21.59) (xy 148.59 21.59)
 		)
 		(stroke
@@
 		)
 	)
+	(global_label "Vref"
+		(shape output)
+		(at 107.95 161.798 0)
+		(fields_autoplaced yes)
+		(effects
+			(font
+				(size 1.27 1.27)
+			)
+			(justify left)
+		)
+		(property "Intersheetrefs" "${INTERSHEET_REFS}"
+			(at 113.9701 161.798 0)
+			(effects
+				(font
+					(size 1.27 1.27)
+				)
+				(justify left)
+				(hide yes)
+			)
+		)
+	)
 	(global_label "SDA"
 		(shape bidirectional)
@@
 		)
 	)
+	(global_label "CE"
+		(shape input)
+		(at 147.574 26.67 180)
+		(fields_autoplaced yes)
+		(effects
+			(font
+				(size 1.27 1.27)
+			)
+			(justify right)
+		)
+		(property "Intersheetrefs" "${INTERSHEET_REFS}"
+			(at 142.824 26.67 0)
+			(effects
+				(font
+					(size 1.27 1.27)
+				)
+				(justify right)
+				(hide yes)
+			)
+		)
+	)
 	(global_label "PWRKEY"
 		(shape output)
@@
 			)
 		)
-		(property "Footprint" "Connector_JST:JST_PH_B2B-PH-K_1x02_P2.00mm_Vertical"
+		(property "Footprint" "Empreintes:1725656"
 			(at 255.016 137.668 0)
 			(effects
@@
 					(unit 1)
 				)
+			)
+		)
+	)
+	(symbol
+		(lib_id "Jumper:SolderJumper_2_Open")
+		(at 76.3 159.07 0)
+		(unit 1)
+		(exclude_from_sim yes)
+		(in_bom no)
+		(on_board yes)
+		(dnp no)
+		(fields_autoplaced yes)
+		(property "Reference" "JP1"
+			(at 76.3 153.68 0)
+			(effects
+				(font
+					(size 1.27 1.27)
+				)
+			)
+		)
+		(property "Value" "SolderJumper_2_Open"
+			(at 76.3 156.22 0)
+			(effects
+				(font
+					(size 1.27 1.27)
+				)
+			)
+		)
+		(property "Footprint" ""
+			(at 76.3 159.07 0)
+			(effects
+				(font
+					(size 1.27 1.27)
+				)
+				(hide yes)
+			)
+		)
+		(property "Datasheet" "~"
+			(at 76.3 159.07 0)
+			(effects
+				(font
+					(size 1.27 1.27)
+				)
+				(hide yes)
+			)
+		)
+		(property "Description" "Solder Jumper, 2-pole, open"
+			(at 76.3 159.07 0)
+			(effects
+				(font
+					(size 1.27 1.27)
+				)
+				(hide yes)
+			)
+		)
+		(pin "2"
+		)
+		(pin "1"
+		)
+		(instances
+			(project "Open_beehive_scale_V0.5"
+				(path "/a4bf92fd-0992-4ef9-a190-19a629782be3"
+					(reference "JP1")
+					(unit 1)
+				)

Commit message: update
Parts:
- J22: footprint Connector_PinHeader_2.54mm:PinHeader_1x08_P2.54mm_Vertical -> Empreintes:Sim8070G
Changed lines of the file:
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@@
 			)
 		)
-		(property "Footprint" "Connector_PinHeader_2.54mm:PinHeader_1x08_P2.54mm_Vertical"
+		(property "Footprint" "Empreintes:Sim8070G"
 			(at 55.88 128.778 0)
 			(effects

Commit message: update
Parts:
- removed JP1: SolderJumper_2_Open, symbol Jumper:SolderJumper_2_Open
- added JP1: Jumper_2_Open, Jumper:SolderJumper-2_P1.3mm_Open_RoundedPad1.0x1.5mm, symbol Jumper:Jumper_2_Open
- J21: footprint Connector_JST:JST_PH_B2B-PH-K_1x02_P2.00mm_Vertical -> Empreintes:1725656
Connections:
- net +5V: now also JP1.1 (A)
- net VCC_MODEM: now also JP1.2 (B)
Changed lines of the file:
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@@
 	)
 	(junction
+		(at 97.92 167.64)
+		(diameter 0)
+		(color 0 0 0 0)
+	)
+	(junction
 		(at 50.8 24.13)
 		(diameter 0)
@@
 	)
 	(junction
+		(at 56.93 167.64)
+		(diameter 0)
+		(color 0 0 0 0)
+	)
+	(junction
 		(at 232.41 78.74)
 		(diameter 0)
@@
 	(wire
 		(pts
+			(xy 56.93 159.59) (xy 56.93 167.64)
+		)
+		(stroke
+			(width 0)
+			(type default)
+		)
+	)
+	(wire
+		(pts
 			(xy 261.62 35.56) (xy 262.89 35.56)
 		)
@@
 	(wire
 		(pts
+			(xy 97.91 159.64) (xy 97.91 159.59)
+		)
+		(stroke
+			(width 0)
+			(type default)
+		)
+	)
+	(wire
+		(pts
 			(xy 156.464 72.644) (xy 156.464 70.104)
 		)
@@
 	(wire
 		(pts
+			(xy 97.91 159.64) (xy 97.92 159.64)
+		)
+		(stroke
+			(width 0)
+			(type default)
+		)
+	)
+	(wire
+		(pts
 			(xy 135.89 123.19) (xy 135.89 130.81)
 		)
@@
 	(wire
 		(pts
-			(xy 91.44 167.64) (xy 102.87 167.64)
+			(xy 91.44 167.64) (xy 97.92 167.64)
+		)
+		(stroke
+			(width 0)
+			(type default)
+		)
+	)
+	(wire
+		(pts
+			(xy 97.92 167.64) (xy 102.87 167.64)
 		)
 		(stroke
@@
 	(wire
 		(pts
-			(xy 45.72 167.64) (xy 63.5 167.64)
+			(xy 45.72 167.64) (xy 56.93 167.64)
 		)
 		(stroke
@@
 	(wire
 		(pts
+			(xy 71.1 159.59) (xy 56.93 159.59)
+		)
+		(stroke
+			(width 0)
+			(type default)
+		)
+	)
+	(wire
+		(pts
 			(xy 182.88 125.73) (xy 187.96 125.73)
 		)
@@
 	(wire
 		(pts
+			(xy 97.91 159.59) (xy 81.26 159.59)
+		)
+		(stroke
+			(width 0)
+			(type default)
+		)
+	)
+	(wire
+		(pts
 			(xy 241.3 78.74) (xy 241.3 80.01)
 		)
@@
 	(wire
 		(pts
+			(xy 56.93 167.64) (xy 63.5 167.64)
+		)
+		(stroke
+			(width 0)
+			(type default)
+		)
+	)
+	(wire
+		(pts
 			(xy 152.4 120.65) (xy 144.78 120.65)
 		)
@@
 	(wire
 		(pts
+			(xy 97.92 167.64) (xy 97.92 159.64)
+		)
+		(stroke
+			(width 0)
+			(type default)
+		)
+	)
+	(wire
+		(pts
 			(xy 130.81 26.67) (xy 130.81 21.59)
 		)
@@
 			)
 		)
-		(property "Footprint" "Connector_JST:JST_PH_B2B-PH-K_1x02_P2.00mm_Vertical"
+		(property "Footprint" "Empreintes:1725656"
 			(at 172.974 84.074 0)
 			(effects
@@
 	)
 	(symbol
-		(lib_id "Jumper:SolderJumper_2_Open")
-		(at 76.3 159.07 0)
-		(unit 1)
-		(exclude_from_sim yes)
-		(in_bom no)
-		(on_board yes)
-		(dnp no)
-		(fields_autoplaced yes)
-		(property "Reference" "JP1"
-			(at 76.3 153.68 0)
-			(effects
-				(font
-					(size 1.27 1.27)
-				)
-			)
-		)
-		(property "Value" "SolderJumper_2_Open"
-			(at 76.3 156.22 0)
-			(effects
-				(font
-					(size 1.27 1.27)
-				)
-			)
-		)
-		(property "Footprint" ""
-			(at 76.3 159.07 0)
-			(effects
-				(font
-					(size 1.27 1.27)
-				)
-				(hide yes)
-			)
-		)
-		(property "Datasheet" "~"
-			(at 76.3 159.07 0)
-			(effects
-				(font
-					(size 1.27 1.27)
-				)
-				(hide yes)
-			)
-		)
-		(property "Description" "Solder Jumper, 2-pole, open"
-			(at 76.3 159.07 0)
-			(effects
-				(font
-					(size 1.27 1.27)
-				)
-				(hide yes)
-			)
-		)
-		(pin "2"
-		)
-		(pin "1"
-		)
-		(instances
-			(project "Open_beehive_scale_V0.5"
-				(path "/a4bf92fd-0992-4ef9-a190-19a629782be3"
-					(reference "JP1")
-					(unit 1)
-				)
-			)
-		)
-	)
-	(symbol
 		(lib_id "Device:C")
 		(at 53.34 66.04 0)
@@
 					(unit 1)
 				)
+			)
+		)
+	)
+	(symbol
+		(lib_id "Jumper:Jumper_2_Open")
+		(at 76.18 159.59 0)
+		(unit 1)
+		(exclude_from_sim yes)
+		(in_bom yes)
+		(on_board yes)
+		(dnp no)
+		(fields_autoplaced yes)
+		(property "Reference" "JP1"
+			(at 76.18 152.4 0)
+			(effects
+				(font
+					(size 1.27 1.27)
+				)
+			)
+		)
+		(property "Value" "Jumper_2_Open"
+			(at 76.18 154.94 0)
+			(effects
+				(font
+					(size 1.27 1.27)
+				)
+			)
+		)
+		(property "Footprint" "Jumper:SolderJumper-2_P1.3mm_Open_RoundedPad1.0x1.5mm"
+			(at 76.18 159.59 0)
+			(effects
+				(font
+					(size 1.27 1.27)
+				)
+				(hide yes)
+			)
+		)
+		(property "Datasheet" "~"
+			(at 76.18 159.59 0)
+			(effects
+				(font
+					(size 1.27 1.27)
+				)
+				(hide yes)
+			)
+		)
+		(property "Description" "Jumper, 2-pole, open"
+			(at 76.18 159.59 0)
+			(effects
+				(font
+					(size 1.27 1.27)
+				)
+				(hide yes)
+			)
+		)
+		(pin "1"
+		)
+		(pin "2"
+		)
+		(instances
+			(project "Open_beehive_scale_V0.5"
+				(path "/a4bf92fd-0992-4ef9-a190-19a629782be3"
+					(reference "JP1")
+					(unit 1)
+				)

Commit message: update
Parts:
- removed JP1: Jumper_2_Open, Jumper:SolderJumper-2_P1.3mm_Open_RoundedPad1.0x1.5mm, symbol Jumper:Jumper_2_Open
- added JP3, JP4: Jumper_2_Open, Jumper:SolderJumper-2_P1.3mm_Open_RoundedPad1.0x1.5mm, symbol Jumper:Jumper_2_Open
Connections:
- net +5V: now also JP4.2 (B)
- net GND: now also J21.1 (Pin_1); no longer J21.2 (Pin_2)
- net Rain_gauge: now also J21.2 (Pin_2); no longer J21.1 (Pin_1)
- net VCC_MODEM: now also JP3.2 (B); no longer J22.8 (Pin_8)
- new net: J22.8 (Pin_8), JP3.1 (A), JP4.1 (A)

Commit message: update
Parts:
- added R44: 100k, Resistor_SMD:R_0603_1608Metric, symbol Device:R
Connections:
- net +5V: now also R44.1
- net CE: now also R44.2
Changed lines of the file:
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@@
 	)
 	(junction
+		(at 146.05 21.59)
+		(diameter 0)
+		(color 0 0 0 0)
+	)
+	(junction
 		(at 104.902 167.64)
 		(diameter 0)
@@
 	)
 	(junction
+		(at 146.05 45.72)
+		(diameter 0)
+		(color 0 0 0 0)
+	)
+	(junction
 		(at 266.7 106.68)
 		(diameter 0)
@@
 	(wire
 		(pts
+			(xy 146.05 21.59) (xy 146.05 34.29)
+		)
+		(stroke
+			(width 0)
+			(type default)
+		)
+	)
+	(wire
+		(pts
 			(xy 91.44 180.34) (xy 91.44 182.88)
 		)
@@
 	(wire
 		(pts
+			(xy 146.05 41.91) (xy 146.05 45.72)
+		)
+		(stroke
+			(width 0)
+			(type default)
+		)
+	)
+	(wire
+		(pts
 			(xy 86.614 138.938) (xy 90.932 138.938)
 		)
@@
 	(wire
 		(pts
+			(xy 146.05 45.72) (xy 148.59 45.72)
+		)
+		(stroke
+			(width 0)
+			(type default)
+		)
+	)
+	(wire
+		(pts
 			(xy 266.7 105.41) (xy 266.7 106.68)
 		)
@@
 	(wire
 		(pts
+			(xy 148.59 45.72) (xy 148.59 26.67)
+		)
+		(stroke
+			(width 0)
+			(type default)
+		)
+	)
+	(wire
+		(pts
 			(xy 229.87 110.49) (xy 248.92 110.49)
 		)
@@
 	(wire
 		(pts
-			(xy 147.574 26.67) (xy 148.59 26.67)
+			(xy 135.89 45.72) (xy 146.05 45.72)
 		)
 		(stroke
@@
 		)
 	)
+	(wire
+		(pts
+			(xy 146.05 21.59) (xy 148.59 21.59)
+		)
+		(stroke
+			(width 0)
+			(type default)
+		)
+	)
 	(polyline
 		(pts
@@
 	(wire
 		(pts
-			(xy 140.97 21.59) (xy 148.59 21.59)
+			(xy 140.97 21.59) (xy 146.05 21.59)
 		)
 		(stroke
@@
 	(global_label "CE"
 		(shape input)
-		(at 147.574 26.67 180)
+		(at 135.89 45.72 180)
 		(fields_autoplaced yes)
 		(effects
@@
 		)
 		(property "Intersheetrefs" "${INTERSHEET_REFS}"
-			(at 142.824 26.67 0)
+			(at 131.14 45.72 0)
 			(effects
 				(font
@@
 					(unit 1)
 				)
+			)
+		)
+	)
+	(symbol
+		(lib_id "Device:R")
+		(at 146.05 38.1 0)
+		(unit 1)
+		(exclude_from_sim no)
+		(in_bom yes)
+		(on_board yes)
+		(dnp no)
+		(property "Reference" "R44"
+			(at 147.828 36.9316 0)
+			(effects
+				(font
+					(size 1.27 1.27)
+				)
+				(justify left)
+			)
+		)
+		(property "Value" "100k"
+			(at 147.828 39.243 0)
+			(effects
+				(font
+					(size 1.27 1.27)
+				)
+				(justify left)
+			)
+		)
+		(property "Footprint" "Resistor_SMD:R_0603_1608Metric"
+			(at 144.272 38.1 90)
+			(effects
+				(font
+					(size 1.27 1.27)
+				)
+				(hide yes)
+			)
+		)
+		(property "Datasheet" "~"
+			(at 146.05 38.1 0)
+			(effects
+				(font
+					(size 1.27 1.27)
+				)
+				(hide yes)
+			)
+		)
+		(property "Description" ""
+			(at 146.05 38.1 0)
+			(effects
+				(font
+					(size 1.27 1.27)
+				)
+				(hide yes)
+			)
+		)
+		(pin "1"
+		)
+		(pin "2"
+		)
+		(instances
+			(project "Open_beehive_scale_V0.5"
+				(path "/a4bf92fd-0992-4ef9-a190-19a629782be3"
+					(reference "R44")
+					(unit 1)
+				)
